Commit message: ino added

File: config/diffbot.ros2_control.xacro (robot description, xacro)
@@ -2,19 +2,8 @@
 <robot xmlns:xacro="http://www.ros.org/wiki/xacro">
   <xacro:macro name="diffbot_ros2_control" params="name">
-    <!-- <xacro:property name="initial_positions" value="${xacro.load_yaml(initial_positions_file)['initial_positions']}"/> -->
     <ros2_control name="${name}" type="system">
-      <!-- <xacro:unless value="${use_mock_hardware}"> -->
         <hardware>
           <plugin>diffbot/DiffBotSystemHardware</plugin>
-          <!-- <param name="zlp">0</param>
-          <param name="example_param_hw_stop_duration_sec">3.0</param> -->
         </hardware>
-      <!-- </xacro:unless> -->
-      <!-- <xacro:if value="${use_mock_hardware}">
-        <hardware>
-          <plugin>mock_components/GenericSystem</plugin>
-          <param name="calculate_dynamics">true</param>
-        </hardware>
-      </xacro:if> -->
       <joint name="left_wheel_joint">
         <command_interface name="velocity"/>

File: config/diffbot.urdf.xacro (robot description, xacro)
@@ -7,4 +7,3 @@
   <xacro:include filename="$(find diffbot)/config/diffbot.ros2_control.xacro" />
   <xacro:diffbot_ros2_control name="DiffBot" />
-  <!-- initial_positions_file="$(arg initial_positions_file)"/> -->
 </robot>

File: config/diffbot_description.urdf.xacro (robot description, xacro)
@@ -3,12 +3,9 @@
   <!-- Constants for robot dimensions -->
   <xacro:property name="PI" value="3.1415926535897931"/>
-  <xacro:property name="base_mass" value="0.3" /> <!-- arbitrary value for base mass -->
   <xacro:property name="base_width" value="0.1" />
   <xacro:property name="base_length" value="0.1" />
   <xacro:property name="base_height" value="0.05" />
-  <xacro:property name="wheel_mass" value="0.3" /> <!-- arbitrary value for wheel mass -->
   <xacro:property name="wheel_len" value="0.020" />
   <xacro:property name="wheel_radius" value="0.015" />
-  <xacro:property name="caster_wheel_mass" value="0.1" /> <!-- arbitrary value for caster wheel mass -->
   <xacro:property name="caster_wheel_radius" value="0.015" />
   <xacro:property name="z_offset" value="-${base_height/2}" /> <!-- Space btw top of beam and the each joint -->
@@ -28,12 +25,4 @@
       <material name="orange"/>
     </visual>
-    <!-- <inertial>
-      <origin xyz="0 0 0" rpy="0 0 0"/>
-      <mass value="${base_mass}"/>
-      <inertia
-        ixx="${base_mass / 12.0 * (base_length*base_length + base_height*base_height)}" ixy="0.0" ixz="0.0"
-        iyy="${base_mass / 12.0 * (base_height*base_height + base_width*base_width)}" iyz="0.0"
-        izz="${base_mass / 12.0 * (base_width*base_width + base_length*base_length)}"/>
-      </inertial> -->
     </link>
     <joint name="left_wheel_joint" type="continuous">
@@ -60,12 +49,4 @@
         <material name="black"/>
       </visual>
-      <!-- <inertial>
-        <origin xyz="0 0 0" rpy="${PI/2} 0 0"/>
-        <mass value="${wheel_mass}"/>
-        <inertia
-          ixx="${wheel_mass / 12.0 * (3*wheel_radius*wheel_radius + wheel_len*wheel_len)}" ixy="0.0" ixz="0.0"
-          iyy="${wheel_mass / 12.0 * (3*wheel_radius*wheel_radius + wheel_len*wheel_len)}" iyz="0.0"
-          izz="${wheel_mass / 2.0 * wheel_radius*wheel_radius}"/>
-        </inertial> -->
       </link>
     <joint name="right_wheel_joint" type="continuous">
@@ -92,12 +73,4 @@
         <material name="black"/>
       </visual>
-      <!-- <inertial>
-        <origin xyz="0 0 0" rpy="${PI/2} 0 0"/>
-        <mass value="${wheel_mass}"/>
-        <inertia
-          ixx="${wheel_mass / 12.0 * (3*wheel_radius*wheel_radius + wheel_len*wheel_len)}" ixy="0.0" ixz="0.0"
-          iyy="${wheel_mass / 12.0 * (3*wheel_radius*wheel_radius + wheel_len*wheel_len)}" iyz="0.0"
-          izz="${wheel_mass / 2.0 * wheel_radius*wheel_radius}"/>
-        </inertial> -->
       </link>
     <joint name="caster_frontal_wheel_joint" type="fixed">
@@ -121,12 +94,4 @@
         <material name="white"/>
       </visual>
-      <!-- <inertial>
-        <origin xyz="0 0 0" rpy="0 0 0"/>
-        <mass value="${caster_wheel_mass}"/>
-        <inertia
-          ixx="${caster_wheel_mass * 0.4 * (caster_wheel_radius * caster_wheel_radius)}" ixy="0.0" ixz="0.0"
-          iyy="${caster_wheel_mass * 0.4 * (caster_wheel_radius * caster_wheel_radius)}" iyz="0.0"
-          izz="${caster_wheel_mass * 0.4 * (caster_wheel_radius * caster_wheel_radius)}"/>
-        </inertial> -->
       </link>
     <joint name="caster_rear_wheel_joint" type="fixed">
@@ -150,12 +115,4 @@
         <material name="white"/>
       </visual>
-      <!-- <inertial>
-        <origin xyz="0 0 0" rpy="0 0 0"/>
-        <mass value="${caster_wheel_mass}"/>
-        <inertia
-          ixx="${caster_wheel_mass * 0.4 * (caster_wheel_radius * caster_wheel_radius)}" ixy="0.0" ixz="0.0"
-          iyy="${caster_wheel_mass * 0.4 * (caster_wheel_radius * caster_wheel_radius)}" iyz="0.0"
-          izz="${caster_wheel_mass * 0.4 * (caster_wheel_radius * caster_wheel_radius)}"/>
-        </inertial> -->
       </link>
 </robot>
